File: hardware/pcb/OpenSmartFocuser/_autosave-OpenSmartFocuser.kicad_sch (KiCad schematic)
At the start: 9 parts, among them J1 Barrel_Jack_Switch, M1 Motor_Servo, U1 NanoS3, U2 TMC2209-LA

Commit message: removed AI readme files
Parts:
- U1: footprint Unexpected Maker:NanoS3 -> OpenSmartFocuser:NanoS3
Changed lines of the file:
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@@
 			)
 		)
-		(property "Footprint" "Unexpected Maker:NanoS3"
+		(property "Footprint" "OpenSmartFocuser:NanoS3"
 			(at 57.15 85.09 0)
 			(effects
